File: pdb.brd (EAGLE design)
At the start: 50 x 100 mm, 53 parts, among them J1 XT60PWFEMALE, Q1 IRFR5305PBF, Q2 IRFR5305PBF, Q3 BSN20,215, Q4 BSN20,215, Q5 BSN20,215, U1 TSR_1-2433, U2 TXB0104, U3 ATMEGA48-20AU, U4 LTC2946CMSPBF, U5 LTC2946CMSPBF, U6 LTC2946CMSPBF, U7 AT30TS74SS8M

Commit message: layout wip
Parts:
- removed A1: D24V50F5SINGLESCREW, jonas_pololu:D24V50F5_SINGLESCREW
- removed JP1, JP3, JP4, JP5, JP6, JP7: (no value), pinhead:1X02
- removed JP2: (no value), pinhead:2X08
- removed JP8: (no value), pinhead:1X03/90
- removed LED_3V: orange, led:CHIP-LED0603
- removed LED_5V: grün, led:CHIP-LED0603
- removed LED_BAT: blau, led:CHIP-LED0603
- removed Q1, Q2: IRFR5305PBF, transistor-power:D-PAK_TO252AA
- removed Q3, Q4, Q5: BSN20,215, jonas_mosfet:BSN20_215
- removed SJ1: (no value), jumper:SJ
- removed U7: AT30TS74SS8M, jonas_microchip:SO08
- removed XTAL1: 20MHz, crystal:HC49UP
- added BAT: XT60PWMALE, amass:XT60PWMALE
- added C10, C11, C12, C15, C16, C18, C19, C20, C22, C8, C9: 100nF, rcl:C0603
- added C13, C14: 47pF, rcl:C0603
- added C17, C21: 4.7µF, rcl:C0603
- added C23: 10µF, rcl:C0603
- added ESC: XT60PWFEMALE, amass:XT60PWFEMALE
- added IC1: FT230XQ, ftdichip:QFN16
- added J2: USB-A, USB:USB-A
- added J3: (no value), adafruit:USB-MINIB
- added L1: 22µH, inductor:IND_TAIYO_NRS6045
- added LED1, LED2, LED3, LED4, LED_RX, LED_TX: (no value), led:CHIP-LED0603
- added R18, R19, R20, R21: 5.6, rcl:R0603
- added R22: 49.9k, rcl:R0603
- added R23: 15.8k, rcl:R0603
- added R24: 10k, rcl:R0603
- added Y1: 16MHz, SparkFun-Clocks:CRYSTAL-SMD-5X3.2-2PAD
- C1, C2: value 100nF -> 330µF; device rcl:C0603 -> rcl:CT7343
- C3: value 22pF -> 47µF
- C4: value 22pF -> 50SVPF18M; device rcl:C0603 -> 50SVPF18M:PCAP_SVP_E7
- C5: value 0,1µF -> 50SVPF18M; device rcl:C0603 -> 50SVPF18M:PCAP_SVP_E7
- C6, C7: value 0,1µF -> 8pF
- D1: value ZD18 -> (none); device diode:DO214BA -> adafruit:SOD-123FL
- ISP: device pinhead:2X03/90 -> pinhead:2X03
- J1: value XT60PWFEMALE -> 1-338068-6; device amass:XT60PWFEMALE -> TE-MicroMatch:CONN_1-338068-6
- R1: value 1k -> 9.53k
- R10, R11: value 10k -> 2m; device rcl:R0603 -> shunt_resistor:3920
- R12: value 10k -> 40m; device rcl:R0603 -> shunt_resistor:BO_CRA2512
- R2: value 10k -> 1.8k
- R3: value 2m -> 10k; device jonas_resistor:3920 -> rcl:R0603
- R4: value 2m -> 5.6; device jonas_resistor:3920 -> rcl:R0603
- R5: value CRA2512-FZ-R040ELF -> 5.6; device jonas_bourns:BO_CRA2512 -> rcl:R0603
- R6: value 1,2k -> 27
- R7: value 250 -> 27
- R8: value 100 -> 4k7
- U1: value TSR_1-2433 -> LMZ13608TZ/NOPBTZA11A-M; device Robo-Lib:TSR-1 -> LMZ13608TZ:TZA11A-M
- U2: value TXB0104 -> ATMEGA2560-16AU100A-M; device jonas_ti:SOP65P640X120-14 -> ATMEGA2560:100A-M
- U3: value ATMEGA48-20AU -> LTC2946CMSPBF; device jonas_atmel:QFP80P900X900X120-32 -> LTC2946:SOP50P489X110-16
- U4, U5: device linear:SOP50P489X110-16 -> LTC2946:SOP50P489X110-16
- U6: value LTC2946CMSPBF -> AOZ1282CI; device linear:SOP50P489X110-16 -> AOZ1282CI:SOT95P280X125-6
- moved C4 115.4 mm to (114.0, 68.0), turned to 90 degrees
- moved U1 106.5 mm to (105.0, 49.0), turned to 180 degrees
- moved U6 101.6 mm to (107.0, 33.0)
- moved R3 95.6 mm to (-35.1, 82.8), turned to 0 degrees
- moved R14 91.5 mm to (-54.8, 83.8), turned to 0 degrees
- moved R15 87.7 mm to (-39.0, 98.0)
- moved R10 87.5 mm to (97.5, 18.0), turned to 0 degrees
- moved R13 87.4 mm to (-54.7, 81.8), turned to 0 degrees
- moved C5 86.6 mm to (105.0, 71.0)
- moved U3 86.6 mm to (97.5, 25.0), turned to 180 degrees
- moved C3 85.5 mm to (89.0, 59.0), turned to 180 degrees
- moved C2 85.0 mm to (91.0, 65.5)
- moved R11 82.5 mm to (93.0, 52.0)
- moved R9 82.1 mm to (14.7, 112.8), turned to 0 degrees
- moved D1 79.2 mm to (102.0, 38.0), turned to 180 degrees
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Connections:
- removed net !ALERT_3V3: U3.25, U6.5
- removed net !ALERT_5V: U3.24, U5.5
- removed net !ALERT_V+: U3.23, U4.5
- removed net !TMP_ALERT: R17.1, U3.32
- removed net AKKU-ZWISCHEN: D1.C, Q1.3, Q2.3, R2.2
- removed net BAT_IN: Q1.4
- removed net EXT_!RST: JP2.16, Q5.3, R12.1
- removed net EXT_3V3: JP2.3, R12.2, R13.2, R14.2, SJ1.2, U2.1
- removed net EXT_A0: JP2.9
- removed net EXT_A3: JP2.7
- removed net EXT_A4: JP2.5
- removed net EXT_D1: JP2.14
- removed net EXT_D2: JP2.12
- removed net EXT_D9: JP2.10
- removed net EXT_SCL_5V: JP2.13
- removed net EXT_SDA_5V: JP2.15
- removed net EXT_SPI_CLK: JP2.11, U2.5
- removed net EXT_SPI_CS: JP2.8, U2.2
- removed net EXT_SPI_MISO: JP2.4, U2.4
- removed net EXT_SPI_MOSI: JP2.6, U2.3
- removed net GPIO1_3V3: U6.3
- removed net GPIO1_5V: U5.3
- removed net GPIO1_V+: U4.3
- removed net GPIO2_3V3: U6.4
- removed net GPIO2_5V: U5.4
- removed net GPIO2_V+: U4.4
- removed net INTVCC_3V3: C7.1, U6.12, U6.14, U6.2
- removed net INTVCC_5V: C6.1, U5.14, U5.2
- removed net INTVCC_V+: C5.1, U4.2
- removed net MISO_5V: ISP.1, R10.1, U3.16
- removed net MOSI_5V: ISP.4, R9.1, U3.15
- removed net N$41: D1.A, Q1.1, Q2.1, R1.2, R2.1
- removed net RESET: ISP.5, U3.29
- removed net RST_H: Q3.1, R15.2, U3.10
- removed net RST_L: Q4.1, R13.1, U3.11
- removed net RX: JP8.2, U3.30
- removed net SCK_5V: ISP.3, R11.1, U3.17
- removed net SENSE+3V3: R5.1, U1.3, U6.16
- removed net SENSE+5V: A1.5, R4.P$1, U5.16
- removed net SENSE+V+: Q2.4, R3.P$1, U4.16
- removed net SS_5V: U2.13, U3.14
- removed net TX: JP8.1, U3.31
- removed net V+: A1.2, J1.POS, JP1.1, JP3.1, R3.P$2, R6.2, U1.1, U4.1, U4.15, U5.1, U6.1
- new net !ALERT_+3V3: R17.1, U2.8, U5.5
- new net !ALERT_+5V: R16.1, U2.7, U4.5
- new net !ALERT_VBAT: R15.1, U2.6, U3.5
- new net !RESET: ISP.5, R3.1, U2.30
- new net +3V3_SENSE+: C23.2, L1.1, R12.1, R22.2, U5.15
- new net +5V_SENSE+: C1.+, C2.+, C3.1, R1.2, R11.P$1, U1.10, U1.11, U4.15
- new net BAT_SENSE+: BAT.POS, R10.P$1, U3.16
- new net FC_!RST: J1.16
- new net FC_CS: J1.8
- new net FC_MISO: J1.4
- new net FC_MOSI: J1.6
- new net FC_SCK: J1.11
- new net FC_SCL: J1.13
- new net FC_SDA: J1.15
- new net MISO: ISP.1, U2.22
- new net MOSI: ISP.4, U2.21
- new net N$10: J3.D+, R6.2
- new net N$12: C18.1, U3.2
- new net N$13: C19.1, U4.14, U4.2
- new net N$14: R21.2, U2.38
- new net N$15: C20.1, U5.12, U5.14, U5.2
- new net N$16: J3.VBUS, R8.2
- new net N$17: R20.2, U2.37
- new net N$18: R19.2, U2.36
- new net N$19: R18.2, U2.35
- new net N$20: LED1.A, R18.1
- new net N$21: LED2.A, R19.1
- new net N$22: LED3.A, R20.1
- new net N$23: LED4.A, R21.1
- new net N$24: R22.1, R23.2, U6.3
- new net N$30: R24.1, U6.4
- new net N$8: LED_TX.C, R4.2
- new net SCK: ISP.3, U2.20
- new net USB_RX: IC1.15, U2.2
- new net USB_TX: IC1.2, U2.3
- new net VBAT: C21.1, C4.1, C5.1, ESC.POS, R10.P$2, R24.2, U1.1, U1.2, U3.1, U3.15, U4.1, U5.1, U6.5
- new net VBUS_SENSE: IC1.12, R8.1, R9.2
- net +3V3: now also J1.3, R12.2, R13.2, R14.2, R15.2, R16.2, R17.2, U5.16; no longer JP6.1, JP7.1, R5.2, R8.2, SJ1.1, U6.15
- net +5V: now also C10.1, C11.1, C12.1, C15.1, C16.1, C17.1, C8.1, C9.1, IC1.1, IC1.10, IC1.8, J1.1, J2.1, LED_RX.A, LED_TX.A, R11.P$2, R3.2, U2.10, U2.100, U2.31, U2.61, U2.80, U2.98, U4.16; no longer C1.1, C2.1, JP2.1, JP4.1, JP5.1, R16.2, R4.P$2, R7.2, U2.14, U3.18, U3.4, U3.6, U5.15, U7.8
- net GND: now also BAT.NEG, C1.-, C10.2, C11.2, C12.2, C13.1, C14.1, C15.2, C16.2, C17.2, C18.2, C19.2, C2.-, C20.2, C21.2, C23.1, C6.1, C7.1, C8.2, C9.2, D1.A, ESC.NEG, IC1.13, IC1.3, J1.2, J2.4, J2.5, J2.6, J3.GND, LED1.C, LED2.C, LED3.C, LED4.C, R2.1, R23.1, R9.1, U1.12, U1.3, U1.5, U1.6, U2.11, U2.32, U2.62, U2.81, U2.99, U3.11, U3.12, U3.14, U3.9, U4.9, U5.9, U6.2; no longer A1.3, A1.4, C1.2, C2.2, C6.2, C7.2, J1.NEG, JP1.2, JP2.2, JP3.2, JP4.2, JP5.2, JP6.2, JP7.2, JP8.3, LED_3V.C, LED_5V.C, LED_BAT.C, Q3.2, Q4.2, R1.1, R15.1, U1.2, U2.7, U3.21, U3.3, U3.5, U4.14, U5.12, U6.11, U7.4
- net N$1: now also R1.1, R2.2, U1.7; no longer R10.2, U2.11
- net N$11: now also J3.D-, R7.1; no longer Q3.3, Q5.2
- net N$2: now also C6.2, U2.34, Y1.P$2; no longer R9.2, U2.12
- net N$27: now also C22.2, D1.C, L1.2, U6.6; no longer C3.1, U3.7, XTAL1.2
- net N$28: now also C22.1, U6.1; no longer C4.1, U3.8, XTAL1.1
- net N$3: now also C7.2, U2.33, Y1.P$1; no longer R11.2, U2.10
- net N$4: now also C13.2, IC1.6; no longer LED_BAT.A
- net N$5: now also C14.2, IC1.7, R7.2; no longer LED_5V.A, R7.1
- net N$6: now also IC1.5, R4.1; no longer R16.1, R17.2, U7.3
- net N$7: now also IC1.11, R5.1; no longer LED_3V.A, R8.1
- net N$9: now also LED_RX.C, R5.2; no longer Q4.3, Q5.1, R14.1
- net SCL: now also R13.1, U2.43, U3.8; no longer U3.28, U6.8, U7.2
- net SDA: now also R14.1, U2.44, U3.6, U3.7; no longer U3.27, U6.6, U6.7, U7.1
Routing:
- net +5V: track 220.5 -> 33.4 mm, vias 6 -> 0
- net V+: track 167.7 -> 0.00 mm, vias 16 -> 0
- net +3V3: track 107.2 -> 8.03 mm, vias 3 -> 0
- net SDA: track 80.4 -> 0.50 mm, vias 5 -> 0
- net SCL: track 77.2 -> 0.00 mm, vias 5 -> 0
- net VBAT: track 0.00 -> 74.5 mm, vias 0 -> 1
- net MOSI_5V: track 58.0 -> 0.00 mm, vias 3 -> 0
- net EXT_3V3: track 52.8 -> 0.00 mm, vias 2 -> 0
- net MISO_5V: track 50.6 -> 0.00 mm, vias 2 -> 0
- net RESET: track 49.3 -> 0.00 mm, vias 2 -> 0
- net SCK_5V: track 46.5 -> 0.00 mm, vias 2 -> 0
- net !ALERT_5V: track 35.9 -> 0.00 mm, vias 2 -> 0
- net !ALERT_V+: track 32.8 -> 0.00 mm, vias 2 -> 0
- net !ALERT_3V3: track 24.8 -> 0.00 mm, vias 2 -> 0
- net RST_H: track 24.1 -> 0.00 mm, vias 2 -> 0
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- added copper zone on layer 1, net +3V3_SENSE+
- added copper zone on layer 1, net +5V_SENSE+
- added copper zone on layer 1, net BAT_SENSE+
- added copper zone on layer 1, net N$27
- added copper zone on layer 1, net VBAT
- removed copper zone on layer 1, net AKKU-ZWISCHEN
- removed copper zone on layer 1, net BAT_IN
- removed copper zone on layer 16, net GND
- removed copper zone on layer 1, net SENSE+V+
- removed copper zone on layer 1, net V+
- removed copper zone on layer 16, net V+
Other:
- board size 50 x 100 mm -> 119 x 114 mm
- board text removed: "3V3"
- board text removed: "5V"
- board text removed: "BAT IN"
- board text removed: "ESC OUT"
- board text removed: "GND"
- board text removed: "RX"
- board text removed: "TX"
- board text removed: "V+"
